File: Qwiic_Quad_Relay.sch (EAGLE design)
At the start: 62 parts, among them J2 Qwiic Right Angle, J3 Qwiic Right Angle, J4 AVR_SPI_PROG_3X2TESTPOINTS, J9 POWER_JACK, K1 RELAY-SPDT-JZC-11F, K2 RELAY-SPDT-JZC-11F, K3 RELAY-SPDT-JZC-11F, K4 RELAY-SPDT-JZC-11F, Q1 600mA/40V, Q2 600mA/40V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

Commit message: Ready for review
Other:
- note removed: "10mA - really close to actual IR on current maybe change to 220?"
- note removed: "205mA - 208mA going to Relay - 133mA Coil Current"
- note removed: "213t"
- note removed: "??"
- note removed: "The board is designed for a 15*C temperature rise Allowing for a continous current draw of 5.5A. The relay can handle 10 A at 110VAC for short pulses (under 20 seconds)."
- note removed: "delay: 10ms for relay and 5ns for Opto-isolator"
- note removed: "w/330 Ohm: All ON: 1.6V dropout ~5mA Single: .4V dropout ~8mA w/220 Ohm 13mA 7mA"
- moved on the sheet: D7, D8, R10, R11, R15, R16, R2, R3, R5, U2, U3

Commit message: Silk, diode, different  LEDs, jumper, rounded route out
I changed to better consistency of label size, a center positive label for the barrel jack, and added the new qwiic label to our new standard. Used different color LEDs so that a person could identify which relay is on by color. I added a jumper to bypass regulator in teh case they use a 5V Wall wart. Finally, I improved the route out - better shape, smaller size.
Parts:
- added D11: 1A/40V/500mV, SparkFun-DiscreteSemi:DIODE-SCHOTTKY-SS14
- added JP7: JUMPER-SMT_2_NO_SILK, SparkFun-Jumpers:JUMPER-SMT_2_NO_SILK
- C4: value 47uF -> 10uF; device SparkFun-Capacitors:47UF-POLAR-EIA3528-10V-10% -> SparkFun-Capacitors:10UF-POLAR-EIA3528-20V-10%(TANT)
- D2: value BLUE -> WHITE; device SparkFun-LED:LED-BLUE0603 -> SparkFun-LED:LED-WHITE0603
- D8: value BLUE -> Yellow; device SparkFun-LED:LED-BLUE0603 -> SparkFun-LED:LED-YELLOW0603
- D9: value BLUE -> GREEN; device SparkFun-LED:LED-BLUE0603 -> SparkFun-LED:LED-GREEN0603
- JP2, JP6, JP8, JP9: value FIDUCIALUFIDUCIAL -> FIDUCIAL1X2; device SparkFun:FIDUCIALUFIDUCIAL -> SparkFun-Aesthetics:FIDUCIAL1X2
Connections:
- new net VIN: D11.A, J9.PWR, JP7.1
- net 5V: now also JP7.2
- net N$4: now also D11.C; no longer J9.PWR
Other:
- note added: "Close Jumper to Bypass Voltage Regulator only if using 5V Power Supply"
- moved on the sheet: D4, D5, D6, D7, D8, D9, J9, K2, K3, K4, Q1, Q2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
