File: Hardware/Qwiic_Quad_Relay.sch (EAGLE design)
At the start: 64 parts, among them J2 Qwiic Right Angle, J3 Qwiic Right Angle, J4 AVR_SPI_PROG_3X2TESTPOINTS, J9 POWER_JACK, K1 RELAY-SPDT-JZC-11F, K2 RELAY-SPDT-JZC-11F, K3 RELAY-SPDT-JZC-11F, K4 RELAY-SPDT-JZC-11F, Q1 600mA/40V, Q2 600mA/40V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

Commit message: Example Code, Firmware, Changes to board
Example Code is not done, firmware as well, unless I want to add a bit more to toggle all channels to opposite states. Production Files have been added. Induction resistor has been changed to a 100 Ohm resistor.
Parts:
- R1, R12, R13, R14: value 10 -> 100; device SparkFun-Resistors:47KOHM-0603-1/10W-1% -> SparkFun-Resistors:100OHM-0603-1/10W-1%
- R8: value 10K -> 10k; device SparkFun-Resistors:330OHM-0603-1/10W-1% -> SparkFun-Resistors:10KOHM-0603-1/10W-1%
- R9: device SparkFun-Resistors:330OHM-0603-1/10W-1% -> SparkFun-Resistors:1KOHM-0603-1/10W-1%
- U1: value V_REG_317SMD -> (none); device SparkFun-IC-Power:V_REG_317SMD -> SparkFun-IC-Power:V_REG_LM1117SOT223
Other:
- note added: "No Address Pin or I2C Jumper"
Changed lines of the file:
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@@
 <part name="GND6" library="SparkFun-PowerSymbols" deviceset="GND" device=""/>
 <part name="SUPPLY7" library="SparkFun-PowerSymbols" deviceset="5V" device="" value="3.3V"/>
-<part name="R1" library="SparkFun-Resistors" deviceset="47KOHM" device="-0603-1/10W-1%" value="10"/>
+<part name="R1" library="SparkFun-Resistors" deviceset="100OHM" device="-0603-1/10W-1%" value="100"/>
 <part name="JP3" library="SparkFun" deviceset="STAND-OFF" device=""/>
 <part name="JP4" library="SparkFun" deviceset="STAND-OFF" device=""/>
@@
 <part name="JP6" library="SparkFun-Aesthetics" deviceset="FIDUCIAL" device="1X2"/>
 <part name="J4" library="SparkFun-Connectors" deviceset="AVR_SPI_PROG_3X2" device="TESTPOINTS"/>
-<part name="R8" library="SparkFun-Resistors" deviceset="330OHM" device="-0603-1/10W-1%" value="10K"/>
-<part name="R9" library="SparkFun-Resistors" deviceset="330OHM" device="-0603-1/10W-1%" value="1k"/>
+<part name="R8" library="SparkFun-Resistors" deviceset="10KOHM" device="-0603-1/10W-1%" value="10k"/>
+<part name="R9" library="SparkFun-Resistors" deviceset="1KOHM" device="-0603-1/10W-1%" value="1k"/>
 <part name="D3" library="SparkFun-LED" deviceset="LED-RED" device="0603" value="RED"/>
 <part name="GND7" library="SparkFun-PowerSymbols" deviceset="GND" device=""/>
@@
 <part name="GND11" library="SparkFun-PowerSymbols" deviceset="GND" device=""/>
 <part name="GND12" library="SparkFun-PowerSymbols" deviceset="GND" device=""/>
-<part name="R12" library="SparkFun-Resistors" deviceset="47KOHM" device="-0603-1/10W-1%" value="10"/>
-<part name="R13" library="SparkFun-Resistors" deviceset="47KOHM" device="-0603-1/10W-1%" value="10"/>
-<part name="R14" library="SparkFun-Resistors" deviceset="47KOHM" device="-0603-1/10W-1%" value="10"/>
+<part name="R12" library="SparkFun-Resistors" deviceset="100OHM" device="-0603-1/10W-1%" value="100"/>
+<part name="R13" library="SparkFun-Resistors" deviceset="100OHM" device="-0603-1/10W-1%" value="100"/>
+<part name="R14" library="SparkFun-Resistors" deviceset="100OHM" device="-0603-1/10W-1%" value="100"/>
 <part name="D7" library="SparkFun-LED" deviceset="LED-BLUE" device="0603" value="BLUE"/>
 <part name="D8" library="SparkFun-LED" deviceset="LED-YELLOW" device="0603" value="Yellow"/>
@@
 <part name="SUPPLY15" library="SparkFun-PowerSymbols" deviceset="5V" device=""/>
 <part name="J9" library="SparkFun-Connectors" deviceset="POWER_JACK" device=""/>
-<part name="U1" library="SparkFun-IC-Power" deviceset="V_REG_317" device="SMD"/>
+<part name="U1" library="SparkFun-IC-Power" deviceset="V_REG_LM1117" device="SOT223"/>
 <part name="GND13" library="SparkFun-PowerSymbols" deviceset="GND" device=""/>
 <part name="R6" library="SparkFun-Resistors" deviceset="240OHM" device="-0603-1/10W-1%" value="240"/>
@@
 <wire x1="134.62" y1="124.46" x2="165.1" y2="124.46" width="0.2032" layer="97" style="shortdash"/>
 <wire x1="165.1" y1="124.46" x2="165.1" y2="106.68" width="0.2032" layer="97" style="shortdash"/>
+<text x="205.74" y="119.38" size="1.778" layer="91">No Address Pin or I2C Jumper</text>
 </plain>
 <instances>

Commit message: Updates to board file, example code, and firmware for release!
Parts:
- R1, R12, R13, R14: value 100 -> 10; device SparkFun-Resistors:100OHM-0603-1/10W-1% -> SparkFun-Resistors:10OHM-0603-1/10W-5%
Changed lines of the file:
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@@
 <part name="GND6" library="SparkFun-PowerSymbols" deviceset="GND" device=""/>
 <part name="SUPPLY7" library="SparkFun-PowerSymbols" deviceset="5V" device="" value="3.3V"/>
-<part name="R1" library="SparkFun-Resistors" deviceset="100OHM" device="-0603-1/10W-1%" value="100"/>
+<part name="R1" library="SparkFun-Resistors" deviceset="10OHM" device="-0603-1/10W-5%" value="10"/>
 <part name="JP3" library="SparkFun" deviceset="STAND-OFF" device=""/>
 <part name="JP4" library="SparkFun" deviceset="STAND-OFF" device=""/>
@@
 <part name="GND11" library="SparkFun-PowerSymbols" deviceset="GND" device=""/>
 <part name="GND12" library="SparkFun-PowerSymbols" deviceset="GND" device=""/>
-<part name="R12" library="SparkFun-Resistors" deviceset="100OHM" device="-0603-1/10W-1%" value="100"/>
-<part name="R13" library="SparkFun-Resistors" deviceset="100OHM" device="-0603-1/10W-1%" value="100"/>
-<part name="R14" library="SparkFun-Resistors" deviceset="100OHM" device="-0603-1/10W-1%" value="100"/>
+<part name="R12" library="SparkFun-Resistors" deviceset="10OHM" device="-0603-1/10W-5%" value="10"/>
+<part name="R13" library="SparkFun-Resistors" deviceset="10OHM" device="-0603-1/10W-5%" value="10"/>
+<part name="R14" library="SparkFun-Resistors" deviceset="10OHM" device="-0603-1/10W-5%" value="10"/>
 <part name="D7" library="SparkFun-LED" deviceset="LED-BLUE" device="0603" value="BLUE"/>
 <part name="D8" library="SparkFun-LED" deviceset="LED-YELLOW" device="0603" value="Yellow"/>

Commit message: Version x02
Changes:
Added thermal polygon around and underneath the voltage regulator.
Changed LED resistor values to 1k because they were too bright.
Added address jumper.
Modified relay pins
Changed Firmware to add second I2C address
Parts:
- added JP10: JUMPER-SMT_2_NO_SILK, SparkFun-Jumpers:JUMPER-SMT_2_NO_SILK
- R15, R16, R17, R4: value 220 -> 1k; device SparkFun-Resistors:220OHM-0603-1/10W-1% -> SparkFun-Resistors:1KOHM-0603-1/10W-1%
Connections:
- new net ADDR_JUMP: JP10.1, U5.(A7)~7
- net GND: now also JP10.2
Other:
- note added: "Address 0x6D: HIGH (Default) Address 0x6C: LOW (Close Jumper)"
- note added: "x02"
- note removed: "No Address Pin or I2C Jumper"
- note removed: "x01"
- moved on the sheet: C1, R8, U5
