File: Hardware/Production/Qwiic_Quad_Relay-Panel.brd (EAGLE design)
At the start: 185.7 x 114.6 mm, 475 parts, among them J10 Qwiic Right Angle, J11 Qwiic Right Angle, J12 AVR_SPI_PROG_3X2TESTPOINTS, J18 POWER_JACK, J19 Qwiic Right Angle, J2 Qwiic Right Angle, J20 Qwiic Right Angle, J21 AVR_SPI_PROG_3X2TESTPOINTS, J27 POWER_JACK, J28 Qwiic Right Angle, J29 Qwiic Right Angle, J3 Qwiic Right Angle, J30 AVR_SPI_PROG_3X2TESTPOINTS, J36 POWER_JACK, J4 AVR_SPI_PROG_3X2TESTPOINTS, J9 POWER_JACK, K1 RELAY-SPDT-JZC-11F, K10 RELAY-SPDT-JZC-11F, K11 RELAY-SPDT-JZC-11F, K12 RELAY-SPDT-JZC-11F, K13 RELAY-SPDT-JZC-11F, K14 RELAY-SPDT-JZC-11F, K15 RELAY-SPDT-JZC-11F, K16 RELAY-SPDT-JZC-11F, K2 RELAY-SPDT-JZC-11F, K3 RELAY-SPDT-JZC-11F, K4 RELAY-SPDT-JZC-11F, K5 RELAY-SPDT-JZC-11F, K6 RELAY-SPDT-JZC-11F, K7 RELAY-SPDT-JZC-11F, K8 RELAY-SPDT-JZC-11F, K9 RELAY-SPDT-JZC-11F, Q1 600mA/40V, Q10 600mA/40V, Q11 600mA/40V, Q12 600mA/40V, Q13 600mA/40V, Q14 600mA/40V, Q15 600mA/40V, Q16 600mA/40V, Q2 600mA/40V, Q3 600mA/40V, Q4 600mA/40V, Q5 600mA/40V, Q6 600mA/40V, Q7 600mA/40V, Q8 600mA/40V, Q9 600mA/40V, U1 V_REG_317SMD, U10 DUAL-OPTOISOLATOR_SOIC8, U11 ATTINY84-ARDUINO, U12 V_REG_317SMD, U13 DUAL-OPTOISOLATOR_SOIC8, U14 DUAL-OPTOISOLATOR_SOIC8, U15 ATTINY84-ARDUINO, U16 V_REG_317SMD, U2 DUAL-OPTOISOLATOR_SOIC8, U3 DUAL-OPTOISOLATOR_SOIC8, U4 DUAL-OPTOISOLATOR_SOIC8, U5 ATTINY84-ARDUINO, U6 DUAL-OPTOISOLATOR_SOIC8, U7 ATTINY84-ARDUINO, U8 V_REG_317SMD, U9 DUAL-OPTOISOLATOR_SOIC8

Commit message: Production Files Updated
Parts:
- added JP37, JP38: FIDUCIAL1X2, SparkFun-Aesthetics:FIDUCIAL-1X2
- added JP39, JP40: JUMPER-SMT_2_NO_SILK, SparkFun-Jumpers:SMT-JUMPER_2_NO_SILK
- added U$225: (no value), qwiic_copyrighted_logo_medium:QWIIC#JPG
- added U$226: (no value), 5V Wall Adapter:5V_WALL_ADAPTER0
- added U$227: (no value), jumper:JUMPER0
- added U$228: (no value), Labels:ADR-()-04
- JP10, JP19, JP20, JP29: value STAND-OFF -> JUMPER-SMT_2_NO_SILK; device SparkFun:STAND-OFF -> SparkFun-Jumpers:SMT-JUMPER_2_NO_SILK
- JP12, JP16, JP21, JP22, JP25, JP26, JP31, JP35: value FIDUCIAL1X2 -> STAND-OFF; device SparkFun-Aesthetics:FIDUCIAL-1X2 -> SparkFun:STAND-OFF
- JP14, JP23, JP24, JP28, JP33: value STAND-OFF -> FIDUCIAL1X2; device SparkFun:STAND-OFF -> SparkFun-Aesthetics:FIDUCIAL-1X2
- JP18, JP27: value JUMPER-SMT_2_NO_SILK -> FIDUCIAL1X2; device SparkFun-Jumpers:SMT-JUMPER_2_NO_SILK -> SparkFun-Aesthetics:FIDUCIAL-1X2
- JP30: value FIDUCIAL1X2 -> JUMPER-SMT_2_NO_SILK; device SparkFun-Aesthetics:FIDUCIAL-1X2 -> SparkFun-Jumpers:SMT-JUMPER_2_NO_SILK
- JP36: value JUMPER-SMT_2_NO_SILK -> STAND-OFF; device SparkFun-Jumpers:SMT-JUMPER_2_NO_SILK -> SparkFun:STAND-OFF
- R15, R16, R17, R19, R30, R31, R32, R36, R4, R47, R48, R49, R53, R64, R65, R66: value 220 -> 1k
- R21, R38, R55, R8: value 10K -> 10k
- U$100, U$103: device 5V:5V0 -> Labels:GND-03
- U$101, U$104: device SDA:SDA0 -> 5V:5V0
- U$102: device Labels:GND-03 -> SDA:SDA0
- U$105: device Labels:SCK-[)-03 -> SDA:SDA0
- U$106, U$220: device Polarity_marking_center_positive#jpg:POLARITY_MARKING_CENTER_POSITIVE#JPG -> Labels:SCK-[)-03
- U$107: device 7-15V:7#15V0 -> Polarity_marking_center_positive#jpg:POLARITY_MARKING_CENTER_POSITIVE#JPG
- U$108: device Polarity_marking_center_positive#jpg:POLARITY_MARKING_CENTER_POSITIVE#JPG -> 7-15V:7#15V0
- U$109, U$166, U$221: device qwiic_copyrighted_logo_medium:QWIIC#JPG -> Polarity_marking_center_positive#jpg:POLARITY_MARKING_CENTER_POSITIVE#JPG
- U$111, U$167: device 5V Wall Adapter:5V_WALL_ADAPTER0 -> qwiic_copyrighted_logo_medium:QWIIC#JPG
- U$112: device jumper:JUMPER0 -> 5V Wall Adapter:5V_WALL_ADAPTER0
- U$113: device Labels:PWR-()-04 -> jumper:JUMPER0
- U$114: device 2:20 -> Labels:ADR-()-04
- U$115: device 1:10 -> Labels:PWR-()-04
- U$116, U$92: device 3:30 -> 2:20
- U$117, U$205: device 4:40 -> 1:10
- U$118, U$150: device Quad:QWIIC_QUAD_0 -> 3:30
- U$119, U$151: device relay:RELAY0 -> 4:40
- U$120: value SPARKX-LOGO4 -> (none); device SparkX:SPARKX-MEDIUM -> Quad:QWIIC_QUAD_0
- U$121: device SparkX:SPARKX-MEDIUM -> relay:RELAY0
- U$122: value (none) -> SPARKX-LOGO4; device NO:NO0 -> SparkX:SPARKX-MEDIUM
- U$123: device COM:COM0 -> SparkX:SPARKX-MEDIUM
- U$124, U$127, U$130, U$133, U$136, U$139, U$142, U$145: device NC:NC0 -> NO:NO0
- U$125, U$128, U$131, U$134, U$137, U$140, U$143: device NO:NO0 -> COM:COM0
- U$126, U$129, U$132, U$135, U$138, U$141, U$144: device COM:COM0 -> NC:NC0
- U$146: device 1:10 -> COM:COM0
- U$147: device 2:20 -> NC:NC0
- U$148, U$60: device 3:30 -> 1:10
- U$149, U$173: device 4:40 -> 2:20
- U$152: device SparkFun-Aesthetics:OSHW-LOGO-S -> Quad:QWIIC_QUAD_0
- U$153: device 7-15V:7#15V0 -> relay:RELAY0
- U$154: device Labels:SCK-[)-03 -> SparkFun-Aesthetics:OSHW-LOGO-S
- U$155: device Labels:GND-03 -> 7-15V:7#15V0
- U$156: device 5V:5V0 -> Labels:SCK-[)-03
- U$157, U$160: device SDA:SDA0 -> Labels:GND-03
- U$158: device Labels:GND-03 -> 5V:5V0
- U$159: device 5V:5V0 -> SDA:SDA0
- U$161: device Labels:SCK-[)-03 -> 5V:5V0
- U$162: device Polarity_marking_center_positive#jpg:POLARITY_MARKING_CENTER_POSITIVE#JPG -> SDA:SDA0
- U$163: device 7-15V:7#15V0 -> Labels:SCK-[)-03
- U$165, U$222: device qwiic_copyrighted_logo_medium:QWIIC#JPG -> 7-15V:7#15V0
- U$168, U$224: device jumper:JUMPER0 -> qwiic_copyrighted_logo_medium:QWIIC#JPG
- U$169: device Labels:PWR-()-04 -> 5V Wall Adapter:5V_WALL_ADAPTER0
- U$170: device 2:20 -> jumper:JUMPER0
- U$171: device 1:10 -> Labels:ADR-()-04
- U$172: device 3:30 -> Labels:PWR-()-04
- U$174: device Quad:QWIIC_QUAD_0 -> 1:10
- U$175, U$207: device relay:RELAY0 -> 3:30
- U$176: value SPARKX-LOGO4 -> (none); device SparkX:SPARKX-MEDIUM -> 4:40
- U$177: device SparkX:SPARKX-MEDIUM -> Quad:QWIIC_QUAD_0
- U$178: device NO:NO0 -> relay:RELAY0
- U$179: value (none) -> SPARKX-LOGO4; device COM:COM0 -> SparkX:SPARKX-MEDIUM
- U$180: device NC:NC0 -> SparkX:SPARKX-MEDIUM
- U$202: device 1:10 -> NO:NO0
- U$203: device 2:20 -> COM:COM0
- U$204: device 3:30 -> NC:NC0
- U$206: device Quad:QWIIC_QUAD_0 -> 2:20
- U$208: device SparkFun-Aesthetics:OSHW-LOGO-S -> 4:40
- U$209: device 7-15V:7#15V0 -> Quad:QWIIC_QUAD_0
- U$210: device Labels:SCK-[)-03 -> relay:RELAY0
- U$211: device Labels:GND-03 -> SparkFun-Aesthetics:OSHW-LOGO-S
- U$212: device 5V:5V0 -> 7-15V:7#15V0
- U$213: device SDA:SDA0 -> Labels:SCK-[)-03
- U$217: device Labels:SCK-[)-03 -> Labels:GND-03
- U$218: device Polarity_marking_center_positive#jpg:POLARITY_MARKING_CENTER_POSITIVE#JPG -> 5V:5V0
- U$219: device 7-15V:7#15V0 -> SDA:SDA0
- U$223: device 5V Wall Adapter:5V_WALL_ADAPTER0 -> Polarity_marking_center_positive#jpg:POLARITY_MARKING_CENTER_POSITIVE#JPG
- U$56: device Labels:PWR-()-04 -> Labels:ADR-()-04
- U$58: device 2:20 -> Labels:PWR-()-04
- U$59: device 1:10 -> 2:20
- U$61, U$93: device 4:40 -> 3:30
- U$62, U$94: device Quad:QWIIC_QUAD_0 -> 4:40
- U$63, U$95: device relay:RELAY0 -> Quad:QWIIC_QUAD_0
- U$64: value SPARKX-LOGO4 -> (none); device SparkX:SPARKX-MEDIUM -> relay:RELAY0
- U$65: value (none) -> SPARKX-LOGO4
- U$66: device NO:NO0 -> SparkX:SPARKX-MEDIUM
- U$67, U$70, U$73, U$76, U$79, U$82, U$85, U$88: device COM:COM0 -> NO:NO0
- U$68, U$71, U$74, U$77, U$80, U$83, U$86, U$89: device NC:NC0 -> COM:COM0
- U$69, U$72, U$75, U$78, U$81, U$84, U$87: device NO:NO0 -> NC:NC0
- U$90: device 1:10 -> NC:NC0
- U$91: device 2:20 -> 1:10
- U$96: device SparkFun-Aesthetics:OSHW-LOGO-S -> relay:RELAY0
- U$97: device 7-15V:7#15V0 -> SparkFun-Aesthetics:OSHW-LOGO-S
- U$98: device Labels:SCK-[)-03 -> 7-15V:7#15V0
- U$99: device Labels:GND-03 -> Labels:SCK-[)-03
- U1, U12, U16, U8: value V_REG_317SMD -> (none)
- moved JP19 151.4 mm to (143.4, 36.4), flipped to the bottom
- moved JP30 123.7 mm to (39.4, 88.6)
- moved U$113 107.4 mm to (147.1, 33.7), flipped to the bottom
- moved U$114 106.0 mm to (124.8, 40.1), flipped to the bottom
- moved JP29 102.9 mm to (60.3, 87.0), flipped to the bottom
- moved U$56 99.1 mm to (41.8, 40.1), flipped to the bottom
- moved JP32 89.6 mm to (163.1, 95.0)
- moved JP23 88.3 mm to (80.0, 92.5), flipped to the bottom
- moved JP22 87.4 mm to (80.0, 95.0), flipped to the top
- moved JP35 85.6 mm to (85.6, 53.1)
- moved JP13 84.6 mm to (163.1, 41.9)
- moved JP17 84.6 mm to (88.1, 2.54)
- moved JP21 77.7 mm to (2.54, 95.0), flipped to the top
- moved JP11 77.5 mm to (85.6, 44.5)
- moved JP15 77.5 mm to (85.6, 2.54)
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Connections:
- new net ADDR_JUMP: JP10.1, U5.6
- new net ADDR_JUMP1: JP20.1, U7.6
- new net ADDR_JUMP2: JP30.1, U11.6
- new net ADDR_JUMP3: JP40.1, U15.6
- net 5V: now also U1.4
- net 5V1: now also JP19.2, U8.4; no longer JP18.2
- net 5V2: now also JP29.2, U12.4; no longer JP27.2
- net 5V3: now also JP39.2, U16.4; no longer JP36.2
- net GND: now also JP10.2
- net GND1: now also JP20.2
- net GND2: now also JP30.2
- net GND3: now also JP40.2
- net VIN1: now also JP19.1; no longer JP18.1
- net VIN2: now also JP29.1; no longer JP27.1
- net VIN3: now also JP39.1; no longer JP36.1
Routing:
- net ADDR_JUMP1: track 0.00 -> 11.0 mm, vias 0 -> 1
- net ADDR_JUMP: track 0.00 -> 11.0 mm, vias 0 -> 1
- net ADDR_JUMP3: track 0.00 -> 11.0 mm, vias 0 -> 1
- net ADDR_JUMP2: track 0.00 -> 11.0 mm, vias 0 -> 1
- net NC9: track 30.8 -> 32.4 mm
- net NC8: track 13.5 -> 15.1 mm
- net NC6: track 23.0 -> 24.5 mm
- net NC4: track 13.5 -> 15.1 mm
- net NC2: track 23.0 -> 24.5 mm
- net NC14: track 23.0 -> 24.5 mm
- net NC10: track 23.0 -> 24.5 mm
- net NC16: track 13.5 -> 15.1 mm
- net NC12: track 13.5 -> 15.1 mm
- net NC1: track 30.8 -> 32.4 mm
- net NC5: track 30.8 -> 32.4 mm
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- added copper zone on layer 1, net 5V
- added copper zone on layer 16, net 5V
- added copper zone on layer 1, net 5V1
- added copper zone on layer 16, net 5V1
- added copper zone on layer 1, net 5V2
- added copper zone on layer 16, net 5V2
- added copper zone on layer 1, net 5V3
- added copper zone on layer 16, net 5V3
Other:
- board size 185.7 x 114.6 mm -> 179.3 x 123.7 mm
- board text added: "x02"
- board text removed: "x01"
